Commit message: rl fixed

File: robots/moborobo/description/robot.udrf.xacro (robot description, xacro)
@@ -1,7 +1,54 @@
 <?xml version="1.0"?>
     <robot xmlns:xacro="http://www.ros.org/wiki/xacro"  name="moborobo_short">
+        <!--
+          All defaults reproduce the stock single-robot description.
+          barn_rl_robot.launch overrides them for multi-robot training.
+          visual           false removes every rendered shape, so the robot is
+                           invisible to cameras and gpu_ray lidars (its own and
+                           other robots').
+          camera           false drops the RGB camera sensor.
+          collide_bitmask  0 leaves Gazebo's default (collides with everything).
+                           Robots given different single bits pass through each
+                           other but still hit the world, whose bitmask is 0xffff.
+          lidar_*          RS-16 vertical sampling and range (urdf/RS-16.urdf.xacro).
+        -->
+        <xacro:arg name="visual"          default="true"/>
+        <xacro:arg name="camera"          default="true"/>
+        <xacro:arg name="collide_bitmask" default="0"/>
+        <xacro:arg name="lidar_v_samples" default="900"/>
+        <xacro:arg name="lidar_v_min"     default="-2.7"/>
+        <xacro:arg name="lidar_v_max"     default="2.7"/>
+        <xacro:arg name="lidar_max_range" default="150.0"/>
         <xacro:include filename="robot_core.xacro" />
         <xacro:include filename="controller.xacro" />
-        <xacro:include filename="camera.xacro"/>
+        <xacro:if value="$(arg camera)">
+            <xacro:include filename="camera.xacro"/>
+        </xacro:if>
         <xacro:include filename="$(find moborobo)/urdf/RS-16.urdf.xacro"/>
+        <xacro:property name="collide_bitmask" value="$(arg collide_bitmask)"/>
+        <xacro:macro name="ghost_collision" params="link">
+            <gazebo reference="${link}">
+                <collision>
+                    <surface>
+                        <contact>
+                            <collide_bitmask>${collide_bitmask}</collide_bitmask>
+                        </contact>
+                    </surface>
+                </collision>
+            </gazebo>
+        </xacro:macro>
+        <xacro:if value="${collide_bitmask != 0}">
+            <xacro:ghost_collision link="base_link"/>
+            <xacro:ghost_collision link="robosense_base_link"/>
+            <xacro:ghost_collision link="front_caster_1"/>
+            <xacro:ghost_collision link="front_caster_2"/>
+            <xacro:ghost_collision link="back_caster_1"/>
+            <xacro:ghost_collision link="back_caster_2"/>
+            <xacro:ghost_collision link="front_wheel_1"/>
+            <xacro:ghost_collision link="front_wheel_2"/>
+            <xacro:ghost_collision link="back_wheel_1"/>
+            <xacro:ghost_collision link="back_wheel_2"/>
+            <xacro:ghost_collision link="left_wheel"/>
+            <xacro:ghost_collision link="right_wheel"/>
+        </xacro:if>
     </robot>

File: robots/moborobo/description/robot_core.xacro (robot description, xacro)
@@ -2,9 +2,9 @@
 <robot xmlns:xacro="http://www.ros.org/wiki/xacro">
     <link name="base_link">
-        <visual>
+        <xacro:if value="$(arg visual)"><visual>
             <geometry>
                 <mesh filename="package://moborobo/meshes/moborobo_short.stl" scale="1 1 1"/>
             </geometry>
-        </visual>
+        </visual></xacro:if>
         <collision>
             <geometry>
@@ -20,5 +20,5 @@
     </link>
     <link name="front_caster_1">
-        <visual>
+        <xacro:if value="$(arg visual)"><visual>
             <geometry>
                 <box size="0.05 0.05 0.05"/>
@@ -27,5 +27,5 @@
                 <color rgba="0.0 0.1 0.0 1"/>
             </material>
-        </visual>
+        </visual></xacro:if>
         <collision>
             <geometry>
@@ -45,11 +45,11 @@
     </joint>
     <link name="front_wheel_1">
-        <visual>
-            <geometry>
-                <cylinder radius="0.04" length="0.0228"/>
-            </geometry>
-            <material name="black">
-            </material>
-        </visual>
+        <xacro:if value="$(arg visual)"><visual>
+            <geometry>
+                <cylinder radius="0.04" length="0.0228"/>
+            </geometry>
+            <material name="black">
+            </material>
+        </visual></xacro:if>
         <collision>
             <geometry>
@@ -69,5 +69,5 @@
     </joint>
     <link name="front_caster_2">
-        <visual>
+        <xacro:if value="$(arg visual)"><visual>
             <geometry>
                 <box size="0.05 0.05 0.05"/>
@@ -76,5 +76,5 @@
                 <color rgba="0.0 0.1 0.0 1"/>
             </material>
-        </visual>
+        </visual></xacro:if>
         <collision>
             <geometry>
@@ -94,11 +94,11 @@
     </joint>
     <link name="front_wheel_2">
-        <visual>
-            <geometry>
-                <cylinder radius="0.04" length="0.0228"/>
-            </geometry>
-            <material name="black">
-            </material>
-        </visual>
+        <xacro:if value="$(arg visual)"><visual>
+            <geometry>
+                <cylinder radius="0.04" length="0.0228"/>
+            </geometry>
+            <material name="black">
+            </material>
+        </visual></xacro:if>
         <collision>
             <geometry>
@@ -118,5 +118,5 @@
     </joint>
     <link name="back_caster_1">
-        <visual>
+        <xacro:if value="$(arg visual)"><visual>
             <geometry>
                 <box size="0.05 0.05 0.05"/>
@@ -125,5 +125,5 @@
                 <color rgba="0.0 0.1 0.0 1"/>
             </material>
-        </visual>
+        </visual></xacro:if>
         <collision>
             <geometry>
@@ -143,11 +143,11 @@
     </joint>
     <link name="back_wheel_1">
-        <visual>
-            <geometry>
-                <cylinder radius="0.04" length="0.0228"/>
-            </geometry>
-            <material name="black">
-            </material>
-        </visual>
+        <xacro:if value="$(arg visual)"><visual>
+            <geometry>
+                <cylinder radius="0.04" length="0.0228"/>
+            </geometry>
+            <material name="black">
+            </material>
+        </visual></xacro:if>
         <collision>
             <geometry>
@@ -167,5 +167,5 @@
     </joint>
     <link name="back_caster_2">
-        <visual>
+        <xacro:if value="$(arg visual)"><visual>
             <geometry>
                 <box size="0.05 0.05 0.05"/>
@@ -174,5 +174,5 @@
                 <color rgba="0.0 0.1 0.0 1"/>
             </material>
-        </visual>
+        </visual></xacro:if>
         <collision>
             <geometry>
@@ -192,11 +192,11 @@
     </joint>
     <link name="back_wheel_2">
-        <visual>
-            <geometry>
-                <cylinder radius="0.04" length="0.0228"/>
-            </geometry>
-            <material name="black">
-            </material>
-        </visual>
+        <xacro:if value="$(arg visual)"><visual>
+            <geometry>
+                <cylinder radius="0.04" length="0.0228"/>
+            </geometry>
+            <material name="black">
+            </material>
+        </visual></xacro:if>
         <collision>
             <geometry>
@@ -216,5 +216,5 @@
     </joint>
 <link name="right_wheel">
-        <visual>
+        <xacro:if value="$(arg visual)"><visual>
             <geometry>
                 <cylinder radius="0.1" length="0.04"/>
@@ -223,5 +223,5 @@
                 <color rgba="0.0 0.0 0.0 1"/>
             </material>
-        </visual>
+        </visual></xacro:if>
         <collision>
             <geometry>
@@ -240,5 +240,5 @@
     </joint>
     <link name="left_wheel">
-        <visual>
+        <xacro:if value="$(arg visual)"><visual>
             <geometry>
                 <cylinder radius="0.1" length="0.04"/>
@@ -247,5 +247,5 @@
                 <color rgba="0.0 0.0 0.0 1"/>
             </material>
-        </visual>
+        </visual></xacro:if>
         <collision>
             <geometry>

File: robots/moborobo/urdf/RS-16.urdf.xacro (robot description, xacro)
@@ -14,10 +14,10 @@
         izz="0.001245079"/>
     </inertial>
-    <visual>
+    <xacro:if value="$(arg visual)"><visual>
       <origin rpy="-1.5707 0 0" xyz="0.005 0 0.53"/>
       <geometry>
         <mesh filename="$(find moborobo)/meshes/robosense_16.dae" scale="0.82 0.82 0.82"/>
       </geometry>
-    </visual>
+    </visual></xacro:if>
     <collision>
       <origin rpy="0 0 0" xyz="0 0 0.53"/>
@@ -54,13 +54,13 @@
             </horizontal>
             <vertical>
-              <samples>900</samples>
+              <samples>$(arg lidar_v_samples)</samples>
               <resolution>1</resolution>
-              <min_angle>-2.7</min_angle>
-              <max_angle>2.7</max_angle>
+              <min_angle>$(arg lidar_v_min)</min_angle>
+              <max_angle>$(arg lidar_v_max)</max_angle>
             </vertical>
           </scan>
           <range>
             <min>0.4</min>
-            <max>150.0</max>
+            <max>$(arg lidar_max_range)</max>
             <resolution>0.001</resolution>
           </range>
@@ -72,8 +72,8 @@
         </ray>
         <plugin name="gazebo_ros_laser_controller" filename="libgazebo_ros_robosense_gpu_laser.so">
-          <topicName>/rs_points</topicName>
+          <topicName>rs_points</topicName>
           <frameName>robosense</frameName>
           <min_range>0.4</min_range>
-          <max_range>150.0</max_range>
+          <max_range>$(arg lidar_max_range)</max_range>
           <gaussianNoise>0.008</gaussianNoise>
         </plugin>
